Commit message: feat(gazebo): add amr_ix1_gazebo package with Ignition Fortress simulation
- Add amr_ix1_gazebo ROS2 package
- Add empty world SDF with physics, lighting, ground plane
- Add gazebo.launch.py with IGN_GAZEBO_RESOURCE_PATH fix
- Configure ros_gz_bridge for /clock and /tf topics
- Successfully spawn AMR-IX1 in Ignition Gazebo 6

File: src/amr_ix1_description/urdf/amr_ix1.urdf.xacro (robot description, xacro)
@@ -293,5 +293,5 @@
     <child  link="cam_stand_Link"/>
     <axis xyz="0 1 0"/>
-    <limit lower="0" upper="-0.7854" effort="10.0" velocity="1.5" />
+    <limit lower="-0.7854" upper="0" effort="10.0" velocity="1.5" />
     <dynamics damping="0.1" friction="0.1"/>
   </joint>

Commit message: feat(gazebo): add ros2_control with diff_drive_controller
- Add gz_ros2_control/GazeboSimSystem hardware interface to URDF
- Configure 4-wheel skid-steer velocity command interfaces
- Add controllers.yaml with diff_drive_controller and joint_state_broadcaster
- Add wheel friction properties (mu1=0.8, mu2=0.6)
- Fix IGN_IP for multicast network warning
- Robot successfully drives with teleop_twist_keyboard

File: src/amr_ix1_description/urdf/amr_ix1.urdf.xacro (robot description, xacro)
@@ -358,3 +358,81 @@
     <child  link="thermal_link"/>
   </joint>
+  <!-- ================================================================
+       ROS2 CONTROL — Hardware Interface
+       Uses ign_ros2_control for Gazebo simulation
+       Same interface will be used for real hardware (ESP32)
+  ================================================================ -->
+  <ros2_control name="amr_ix1_system" type="system">
+    <hardware>
+      <plugin>gz_ros2_control/GazeboSimSystem</plugin>
+    </hardware>
+    <!-- Front Right Wheel -->
+    <joint name="F_R_W_joint">
+      <command_interface name="velocity">
+        <param name="min">-10</param>
+        <param name="max">10</param>
+      </command_interface>
+      <state_interface name="position"/>
+      <state_interface name="velocity"/>
+    </joint>
+    <!-- Front Left Wheel -->
+    <joint name="F_L_W_joint">
+      <command_interface name="velocity">
+        <param name="min">-10</param>
+        <param name="max">10</param>
+      </command_interface>
+      <state_interface name="position"/>
+      <state_interface name="velocity"/>
+    </joint>
+    <!-- Back Right Wheel -->
+    <joint name="B_R_W_joint">
+      <command_interface name="velocity">
+        <param name="min">-10</param>
+        <param name="max">10</param>
+      </command_interface>
+      <state_interface name="position"/>
+      <state_interface name="velocity"/>
+    </joint>
+    <!-- Back Left Wheel -->
+    <joint name="B_L_W_joint">
+      <command_interface name="velocity">
+        <param name="min">-10</param>
+        <param name="max">10</param>
+      </command_interface>
+      <state_interface name="position"/>
+      <state_interface name="velocity"/>
+    </joint>
+  </ros2_control>
+  <!-- Gazebo plugin to load ign_ros2_control -->
+  <gazebo>
+    <plugin name="gz_ros2_control::GazeboSimROS2ControlPlugin"
+        filename="libgz_ros2_control-system.so">
+      <parameters>$(find amr_ix1_gazebo)/config/controllers.yaml</parameters>
+    </plugin>
+  </gazebo>
+  <!-- Wheel friction properties for Gazebo -->
+  <gazebo reference="F_R_W_Link">
+    <mu1>0.8</mu1>
+    <mu2>0.6</mu2>
+    <kp>1000000.0</kp>
+    <kd>1.0</kd>
+  </gazebo>
+  <gazebo reference="F_L_W_Link">
+    <mu1>0.8</mu1>
+    <mu2>0.6</mu2>
+    <kp>1000000.0</kp>
+    <kd>1.0</kd>
+  </gazebo>
+  <gazebo reference="B_R_W_Link">
+    <mu1>0.8</mu1>
+    <mu2>0.6</mu2>
+    <kp>1000000.0</kp>
+    <kd>1.0</kd>
+  </gazebo>
+  <gazebo reference="B_L_W_Link">
+    <mu1>0.8</mu1>
+    <mu2>0.6</mu2>
+    <kp>1000000.0</kp>
+    <kd>1.0</kd>
+  </gazebo>
 </robot>

Commit message: feat(sensors): add LiDAR sensor plugin and ros2_control integration
- Add gpu_lidar sensor to laser_Link in URDF
- Add gz_ros2_control/GazeboSimSystem hardware interface
- Configure diff_drive_controller for 4-wheel skid-steer
- Add joint_state_broadcaster for all joint states
- Add wheel friction properties (mu1=0.8, mu2=0.6)
- Add RViz to gazebo launch file
- LiDAR publishing at ~4Hz on /lidar topic
- All 11 TF links OK with odom fixed frame
- Robot drives and laser scan visible in RViz

File: src/amr_ix1_description/urdf/amr_ix1.urdf.xacro (robot description, xacro)
@@ -403,4 +403,13 @@
       <state_interface name="velocity"/>
     </joint>
+    <!-- Camera Stand — position controlled -->
+    <joint name="cam_stand_joint">
+      <command_interface name="position">
+        <param name="min">-0.7854</param>
+        <param name="max">0.0</param>
+      </command_interface>
+      <state_interface name="position"/>
+      <state_interface name="velocity"/>
+    </joint>
   </ros2_control>
   <!-- Gazebo plugin to load ign_ros2_control -->
@@ -436,3 +445,42 @@
     <kd>1.0</kd>
   </gazebo>
+  <!-- ================================================================
+       LIDAR SENSOR — RPLidar A2 (simulated)
+       Mounted on laser_Link
+  ================================================================ -->
+  <gazebo reference="laser_Link">
+    <sensor name="gpu_lidar" type="gpu_lidar">
+      <topic>lidar</topic>
+      <gz_frame_id>laser_Link</gz_frame_id>
+      <update_rate>10</update_rate>
+      <ray>
+        <scan>
+          <horizontal>
+            <samples>360</samples>
+            <resolution>1</resolution>
+            <min_angle>-3.14159</min_angle>
+            <max_angle>3.14159</max_angle>
+          </horizontal>
+          <vertical>
+            <samples>1</samples>
+            <resolution>0.01</resolution>
+            <min_angle>0</min_angle>
+            <max_angle>0</max_angle>
+          </vertical>
+        </scan>
+        <range>
+          <min>0.15</min>
+          <max>12.0</max>
+          <resolution>0.01</resolution>
+        </range>
+        <noise>
+          <type>gaussian</type>
+          <mean>0.0</mean>
+          <stddev>0.01</stddev>
+        </noise>
+      </ray>
+      <always_on>1</always_on>
+      <visualize>true</visualize>
+    </sensor>
+  </gazebo>
 </robot>

Commit message: feat(sensors): complete sensor suite + switch to empty world for SLAM
- IMU, RGB camera, thermal camera all publishing
- Factory world preserved for future use
- Switched launch to empty world for SLAM development
- Collision mesh issue logged for Blender fix

File: src/amr_ix1_description/urdf/amr_ix1.urdf.xacro (robot description, xacro)
@@ -89,5 +89,5 @@
   </link>
   <joint name="F_R_W_joint" type="continuous">
-    <origin xyz="0.273978 -0.529050 -0.259730" rpy="0 0 0"/>
+    <origin xyz="0.36129 -0.53208 -0.26273" rpy="0 0 0"/>
     <parent link="base_link"/>
     <child  link="F_R_W_Link"/>
@@ -124,5 +124,5 @@
   </link>
   <joint name="F_L_W_joint" type="continuous">
-    <origin xyz="0.272414 0.541050 -0.262472" rpy="0 0 0"/>
+    <origin xyz="0.35973 0.53802 -0.26547" rpy="0 0 0"/>
     <parent link="base_link"/>
     <child  link="F_L_W_Link"/>
@@ -159,5 +159,5 @@
   </link>
   <joint name="B_R_W_joint" type="continuous">
-    <origin xyz="-0.444885 -0.528950 -0.259725" rpy="0 0 0"/>
+    <origin xyz="-0.35757 -0.53198 -0.26273" rpy="0 0 0"/>
     <parent link="base_link"/>
     <child  link="B_R_W_Link"/>
@@ -194,5 +194,5 @@
   </link>
   <joint name="B_L_W_joint" type="continuous">
-    <origin xyz="-0.446680 0.541050 -0.256487" rpy="0 0 0"/>
+    <origin xyz="-0.35936 0.53802 -0.25949" rpy="0 0 0"/>
     <parent link="base_link"/>
     <child  link="B_L_W_Link"/>
@@ -258,5 +258,5 @@
   </link>
   <joint name="laser_joint" type="fixed">
-    <origin xyz="0.328135 -0.004554 0.047500" rpy="0 0 0"/>
+    <origin xyz="0.41545 -0.0075875 0.0445" rpy="0 0 0"/>
     <parent link="base_link"/>
     <child  link="laser_Link"/>
@@ -289,5 +289,5 @@
   </link>
   <joint name="cam_stand_joint" type="revolute">
-    <origin xyz="-0.274040 -0.063863 0.520470" rpy="0 0 0"/>
+    <origin xyz="-0.18673 -0.066896 0.51747" rpy="0 0 0"/>
     <parent link="base_link"/>
     <child  link="cam_stand_Link"/>
@@ -365,5 +365,5 @@
   <ros2_control name="amr_ix1_system" type="system">
     <hardware>
-      <plugin>gz_ros2_control/GazeboSimSystem</plugin>
+      <plugin>ign_ros2_control/IgnitionSystem</plugin>
     </hardware>
     <!-- Front Right Wheel -->
@@ -415,6 +415,5 @@
   <!-- Gazebo plugin to load ign_ros2_control -->
   <gazebo>
-    <plugin name="gz_ros2_control::GazeboSimROS2ControlPlugin"
-        filename="libgz_ros2_control-system.so">
+    <plugin filename="libign_ros2_control-system.so" name="ign_ros2_control::IgnitionROS2ControlPlugin">
       <parameters>$(find amr_ix1_gazebo)/config/controllers.yaml</parameters>
     </plugin>
@@ -457,5 +456,5 @@
         <scan>
           <horizontal>
-            <samples>360</samples>
+            <samples>180</samples>
             <resolution>1</resolution>
             <min_angle>-3.14159</min_angle>
@@ -481,5 +480,5 @@
       </ray>
       <always_on>1</always_on>
-      <visualize>true</visualize>
+      <visualize>false</visualize>
     </sensor>
   </gazebo>
@@ -491,5 +490,5 @@
     <sensor name="imu_sensor" type="imu">
       <always_on>true</always_on>
-      <update_rate>100</update_rate>
+      <update_rate>50</update_rate>
       <visualize>true</visualize>
       <topic>imu</topic>
@@ -551,5 +550,5 @@
       <gz_frame_id>camera_Link</gz_frame_id>
       <always_on>true</always_on>
-      <update_rate>30</update_rate>
+      <update_rate>10</update_rate>
       <visualize>true</visualize>
       <camera>
@@ -582,6 +581,6 @@
       <gz_frame_id>thermal_link</gz_frame_id>
       <always_on>true</always_on>
-      <update_rate>9</update_rate>
-      <visualize>true</visualize>
+      <update_rate>5</update_rate>
+      <visualize>false</visualize>
       <camera>
         <horizontal_fov>0.9599</horizontal_fov>
@@ -595,6 +594,30 @@
           <far>30</far>
         </clip>
+        <!-- Temperature range: 0=300K(cold/black), 255=400K(hot/white) -->
+        <min_temp>300.0</min_temp>
+        <max_temp>400.0</max_temp>
       </camera>
     </sensor>
   </gazebo>
+  <!-- ================================================================
+       THERMAL PROPERTIES — required for thermal camera sensor
+  ================================================================ -->
+  <gazebo reference="base_link">
+    <temperature>310.0</temperature>
+  </gazebo>
+  <gazebo reference="F_R_W_Link">
+    <temperature>305.0</temperature>
+  </gazebo>
+  <gazebo reference="F_L_W_Link">
+    <temperature>305.0</temperature>
+  </gazebo>
+  <gazebo reference="B_R_W_Link">
+    <temperature>305.0</temperature>
+  </gazebo>
+  <gazebo reference="B_L_W_Link">
+    <temperature>305.0</temperature>
+  </gazebo>
+  <gazebo reference="laser_Link">
+    <temperature>308.0</temperature>
+  </gazebo>
 </robot>

Commit message: fix(navigation): connect Nav2 cmd_vel to diff_drive_controller via twist_stamper
- Add twist_stamper node to bridge Twist -> TwistStamped
- Fix cmd_vel topic mismatch between Nav2 velocity_smoother and diff_drive_controller
- Switch wheel collisions to spheres for performance
- Lighten factory world via Blender re-export, add simplified collision mesh
- Add amr_ix1_navigation package (Nav2 bringup, factory_map)
- Add amr_ix1_slam package (kept for reference)
- Remove tracked .blend files (now gitignored)
- Confirmed robot drives autonomously toward Nav2 goals in factory world

File: src/amr_ix1_description/urdf/amr_ix1.urdf.xacro (robot description, xacro)
@@ -39,5 +39,5 @@
   <link name="base_link">
     <inertial>
-      <origin xyz="-0.048088 0.015216 -0.117965" rpy="0 0 0"/>
+      <origin xyz="0.0 0.0 0.0" rpy="0 0 0"/>
       <mass value="17.7024"/>
       <inertia
@@ -54,7 +54,7 @@
     </visual>
     <collision>
-      <origin xyz="0 0 0" rpy="0 0 0"/>
-      <geometry>
-        <mesh filename="package://amr_ix1_description/meshes/collision/base_link.STL"/>
+      <origin xyz="0 0 0.05" rpy="0 0 0"/>
+      <geometry>
+        <box size="0.60 0.40 0.20"/>
       </geometry>
     </collision>
@@ -65,10 +65,7 @@
   <link name="F_R_W_Link">
     <inertial>
-      <origin xyz="0.000654 0.055120 0.000386" rpy="0 0 0"/>
-      <mass value="5.1478"/>
-      <inertia
-        ixx="0.035042" ixy="2.794E-11" ixz="-7.220E-05"
-        iyy="0.058291"  iyz="-7.127E-11"
-        izz="0.035111"/>
+      <origin rpy="0 0 0" xyz="0 0 0"/>
+      <mass value="1.5"/>
+      <inertia ixx="0.0029" ixy="0.0" ixz="0.0" iyy="0.0029" iyz="0.0" izz="0.0042"/>
     </inertial>
     <visual>
@@ -83,6 +80,5 @@
       <origin xyz="0 0 0" rpy="0 0 0"/>
       <geometry>
-        <mesh filename="package://amr_ix1_description/meshes/collision/F_R_W_Link.STL"/>
-              <scale>0.001 0.001 0.001</scale>
+        <sphere radius="0.15"/>
       </geometry>
     </collision>
@@ -93,5 +89,5 @@
     <child  link="F_R_W_Link"/>
     <axis xyz="0 1 0"/>
-    <dynamics damping="0.1" friction="0.1"/>
+    <dynamics damping="0.2" friction="0.2"/>
   </joint>
   <!-- ================================================================
@@ -100,10 +96,7 @@
   <link name="F_L_W_Link">
     <inertial>
-      <origin xyz="5.723E-07 -0.055120 -0.000759" rpy="0 0 0"/>
-      <mass value="5.1478"/>
-      <inertia
-        ixx="0.035156" ixy="-7.557E-11" ixz="-4.648E-06"
-        iyy="0.058291"  iyz="-1.223E-11"
-        izz="0.034997"/>
+      <origin rpy="0 0 0" xyz="0 0 0"/>
+      <mass value="1.5"/>
+      <inertia ixx="0.0029" ixy="0.0" ixz="0.0" iyy="0.0029" iyz="0.0" izz="0.0042"/>
     </inertial>
     <visual>
@@ -118,6 +111,5 @@
       <origin xyz="0 0 0" rpy="0 0 0"/>
       <geometry>
-        <mesh filename="package://amr_ix1_description/meshes/collision/F_L_W_Link.STL"/>
-              <scale>0.001 0.001 0.001</scale>
+        <sphere radius="0.15"/>
       </geometry>
     </collision>
@@ -128,5 +120,5 @@
     <child  link="F_L_W_Link"/>
     <axis xyz="0 1 0"/>
-    <dynamics damping="0.1" friction="0.1"/>
+    <dynamics damping="0.2" friction="0.2"/>
   </joint>
   <!-- ================================================================
@@ -135,10 +127,7 @@
   <link name="B_R_W_Link">
     <inertial>
-      <origin xyz="-9.003E-06 0.055120 -0.000759" rpy="0 0 0"/>
-      <mass value="5.1478"/>
-      <inertia
-        ixx="0.035157" ixy="-7.543E-11" ixz="2.874E-06"
-        iyy="0.058291"  iyz="1.306E-11"
-        izz="0.034997"/>
+      <origin rpy="0 0 0" xyz="0 0 0"/>
+      <mass value="1.5"/>
+      <inertia ixx="0.0029" ixy="0.0" ixz="0.0" iyy="0.0029" iyz="0.0" izz="0.0042"/>
     </inertial>
     <visual>
@@ -153,6 +142,5 @@
       <origin xyz="0 0 0" rpy="0 0 0"/>
       <geometry>
-        <mesh filename="package://amr_ix1_description/meshes/collision/B_R_W_Link.STL"/>
-              <scale>0.001 0.001 0.001</scale>
+        <sphere radius="0.15"/>
       </geometry>
     </collision>
@@ -163,5 +151,5 @@
     <child  link="B_R_W_Link"/>
     <axis xyz="0 1 0"/>
-    <dynamics damping="0.1" friction="0.1"/>
+    <dynamics damping="0.2" friction="0.2"/>
   </joint>
   <!-- ================================================================
@@ -170,10 +158,7 @@
   <link name="B_L_W_Link">
     <inertial>
-      <origin xyz="-0.000649 -0.055120 0.000395" rpy="0 0 0"/>
-      <mass value="5.1478"/>
-      <inertia
-        ixx="0.035044" ixy="2.886E-11" ixz="7.307E-05"
-        iyy="0.058291"  iyz="7.090E-11"
-        izz="0.035109"/>
+      <origin rpy="0 0 0" xyz="0 0 0"/>
+      <mass value="1.5"/>
+      <inertia ixx="0.0029" ixy="0.0" ixz="0.0" iyy="0.0029" iyz="0.0" izz="0.0042"/>
     </inertial>
     <visual>
@@ -188,6 +173,5 @@
       <origin xyz="0 0 0" rpy="0 0 0"/>
       <geometry>
-        <mesh filename="package://amr_ix1_description/meshes/collision/B_L_W_Link.STL"/>
-              <scale>0.001 0.001 0.001</scale>
+        <sphere radius="0.15"/>
       </geometry>
     </collision>
@@ -198,5 +182,5 @@
     <child  link="B_L_W_Link"/>
     <axis xyz="0 1 0"/>
-    <dynamics damping="0.1" friction="0.1"/>
+    <dynamics damping="0.2" friction="0.2"/>
   </joint>
   <!-- ================================================================
@@ -421,29 +405,37 @@
   <!-- Wheel friction properties for Gazebo -->
   <gazebo reference="F_R_W_Link">
-    <mu1>0.8</mu1>
-    <mu2>0.6</mu2>
-    <kp>1000000.0</kp>
-    <kd>1.0</kd>
+    <mu1>1.0</mu1>
+    <mu2>0.05</mu2>
+    <fdir1>1 0 0</fdir1>
+    <kp>100000.0</kp>
+    <kd>100.0</kd>
+    <minDepth>0.001</minDepth>
   </gazebo>
   <gazebo reference="F_L_W_Link">
-    <mu1>0.8</mu1>
-    <mu2>0.6</mu2>
-    <kp>1000000.0</kp>
-    <kd>1.0</kd>
+    <mu1>1.0</mu1>
+    <mu2>0.05</mu2>
+    <fdir1>1 0 0</fdir1>
+    <kp>100000.0</kp>
+    <kd>100.0</kd>
+    <minDepth>0.001</minDepth>
   </gazebo>
   <gazebo reference="B_R_W_Link">
-    <mu1>0.8</mu1>
-    <mu2>0.6</mu2>
-    <kp>1000000.0</kp>
-    <kd>1.0</kd>
+    <mu1>1.0</mu1>
+    <mu2>0.05</mu2>
+    <fdir1>1 0 0</fdir1>
+    <kp>100000.0</kp>
+    <kd>100.0</kd>
+    <minDepth>0.001</minDepth>
   </gazebo>
   <gazebo reference="B_L_W_Link">
-    <mu1>0.8</mu1>
-    <mu2>0.6</mu2>
-    <kp>1000000.0</kp>
-    <kd>1.0</kd>
-  </gazebo>
-  <!-- ================================================================
-       LIDAR SENSOR — RPLidar A2 (simulated)
+    <mu1>1.0</mu1>
+    <mu2>0.05</mu2>
+    <fdir1>1 0 0</fdir1>
+    <kp>100000.0</kp>
+    <kd>100.0</kd>
+    <minDepth>0.001</minDepth>
+  </gazebo>
+  <!-- ================================================================
+       LIDAR SENSOR — RPLidar A1 (simulated)
        Mounted on laser_Link
   ================================================================ -->
@@ -452,12 +444,12 @@
       <topic>lidar</topic>
       <gz_frame_id>laser_Link</gz_frame_id>
-      <update_rate>10</update_rate>
+      <update_rate>20</update_rate>
       <ray>
         <scan>
           <horizontal>
-            <samples>180</samples>
+            <samples>360</samples>
             <resolution>1</resolution>
-            <min_angle>-3.14159</min_angle>
-            <max_angle>3.14159</max_angle>
+            <min_angle>-2.9</min_angle>
+            <max_angle>2.9</max_angle>
           </horizontal>
           <vertical>
@@ -469,5 +461,5 @@
         </scan>
         <range>
-          <min>0.15</min>
+          <min>0.2</min>
           <max>12.0</max>
           <resolution>0.01</resolution>
@@ -480,5 +472,5 @@
       </ray>
       <always_on>1</always_on>
-      <visualize>false</visualize>
+      <visualize>true</visualize>
     </sensor>
   </gazebo>
