Commit message: fix(navigation): correct robot footprint, inflation radius, and initial pose
- Fix Nav2 footprint from assumed 1.1x1.1m square to real 0.84x1.02m rectangle
  based on actual URDF wheel joint positions (wheel_x=0.36, wheel_y=0.45, radius=0.155)
- Fix inflation_radius from 0.5 to 0.45 to match inscribed radius of corrected footprint
- Remove broken default_nav_through_poses_bt_xml reference from nav2_params.yaml
- Fix inspection_mission.py INITIAL_POSE quaternion (z=0.40 was invalid, corrected to z=0.0)
- Add map_server yaml_filename comment clarifying it is overridden by launch argument

File: src/amr_ix1_description/urdf/amr_ix1.urdf.xacro (robot description, xacro)
@@ -54,7 +54,7 @@
     </visual>
     <collision>
-      <origin xyz="0 0 0.05" rpy="0 0 0"/>
-      <geometry>
-        <box size="0.60 0.40 0.20"/>
+      <origin xyz="0.10 0 0.11" rpy="0 0 0"/>
+      <geometry>
+        <box size="0.90 0.75 0.25"/>
       </geometry>
     </collision>
@@ -78,16 +78,16 @@
     </visual>
     <collision>
-      <origin xyz="0 0 0" rpy="0 0 0"/>
-      <geometry>
-        <sphere radius="0.15"/>
-      </geometry>
+	  <origin xyz="0 -0.025 0" rpy="1.5708 0 0"/>
+	  <geometry>
+	    <cylinder radius="0.155" length="0.12"/>
+	  </geometry>
     </collision>
   </link>
   <joint name="F_R_W_joint" type="continuous">
-    <origin xyz="0.36129 -0.53208 -0.26273" rpy="0 0 0"/>
+    <origin xyz="0.36 -0.45 -0.0300" rpy="0 0 0"/>
     <parent link="base_link"/>
     <child  link="F_R_W_Link"/>
     <axis xyz="0 1 0"/>
-    <dynamics damping="0.2" friction="0.2"/>
+    <dynamics damping="3.0" friction="2.0"/>
   </joint>
   <!-- ================================================================
@@ -109,16 +109,16 @@
     </visual>
     <collision>
-      <origin xyz="0 0 0" rpy="0 0 0"/>
-      <geometry>
-        <sphere radius="0.15"/>
-      </geometry>
+	  <origin xyz="0 0.025 0" rpy="1.5708 0 0"/>
+	  <geometry>
+	    <cylinder radius="0.155" length="0.12"/>
+	  </geometry>
     </collision>
   </link>
   <joint name="F_L_W_joint" type="continuous">
-    <origin xyz="0.35973 0.53802 -0.26547" rpy="0 0 0"/>
+    <origin xyz="0.36 0.45 -0.0300" rpy="0 0 0"/>
     <parent link="base_link"/>
     <child  link="F_L_W_Link"/>
     <axis xyz="0 1 0"/>
-    <dynamics damping="0.2" friction="0.2"/>
+    <dynamics damping="3.0" friction="2.0"/>
   </joint>
   <!-- ================================================================
@@ -140,16 +140,16 @@
     </visual>
     <collision>
-      <origin xyz="0 0 0" rpy="0 0 0"/>
-      <geometry>
-        <sphere radius="0.15"/>
-      </geometry>
+	  <origin xyz="0 -0.025 0" rpy="1.5708 0 0"/>
+	  <geometry>
+	    <cylinder radius="0.155" length="0.12"/>
+	  </geometry>
     </collision>
   </link>
   <joint name="B_R_W_joint" type="continuous">
-    <origin xyz="-0.35757 -0.53198 -0.26273" rpy="0 0 0"/>
+    <origin xyz="-0.36 -0.45 -0.0300" rpy="0 0 0"/>
     <parent link="base_link"/>
     <child  link="B_R_W_Link"/>
     <axis xyz="0 1 0"/>
-    <dynamics damping="0.2" friction="0.2"/>
+    <dynamics damping="3.0" friction="2.0"/>
   </joint>
   <!-- ================================================================
@@ -171,16 +171,16 @@
     </visual>
     <collision>
-      <origin xyz="0 0 0" rpy="0 0 0"/>
-      <geometry>
-        <sphere radius="0.15"/>
-      </geometry>
+	  <origin xyz="0 0.025 0" rpy="1.5708 0 0"/>
+	  <geometry>
+	    <cylinder radius="0.155" length="0.12"/>
+	  </geometry>
     </collision>
   </link>
   <joint name="B_L_W_joint" type="continuous">
-    <origin xyz="-0.35936 0.53802 -0.25949" rpy="0 0 0"/>
+    <origin xyz="-0.36 0.45 -0.0300" rpy="0 0 0"/>
     <parent link="base_link"/>
     <child  link="B_L_W_Link"/>
     <axis xyz="0 1 0"/>
-    <dynamics damping="0.2" friction="0.2"/>
+    <dynamics damping="3.0" friction="2.0"/>
   </joint>
   <!-- ================================================================
@@ -197,5 +197,5 @@
     </inertial>
     <visual>
-      <origin xyz="0 0 0" rpy="0 0 0"/>
+      <origin xyz="0 0 0" rpy="3.14159 0 0"/>
       <geometry>
         <mesh filename="package://amr_ix1_description/meshes/visual/imu_Link.STL"/>
@@ -204,5 +204,5 @@
     </visual>
     <collision>
-      <origin xyz="0 0 0" rpy="0 0 0"/>
+      <origin xyz="0 0 0" rpy="3.14159 0 0"/>
       <geometry>
         <mesh filename="package://amr_ix1_description/meshes/collision/imu_Link.STL"/>
@@ -211,5 +211,5 @@
   </link>
   <joint name="imu_joint" type="fixed">
-    <origin xyz="0.000249 0.003020 -0.012600" rpy="0 0 0"/>
+    <origin xyz="0.0 0.0 0.0" rpy="0 0 0"/>
     <parent link="base_link"/>
     <child  link="imu_Link"/>
@@ -242,5 +242,5 @@
   </link>
   <joint name="laser_joint" type="fixed">
-    <origin xyz="0.41545 -0.0075875 0.0445" rpy="0 0 0"/>
+    <origin xyz="0.415447680695362 -0.00758871084657819 0.27756000072765" rpy="0 0 0"/>
     <parent link="base_link"/>
     <child  link="laser_Link"/>
@@ -273,5 +273,5 @@
   </link>
   <joint name="cam_stand_joint" type="revolute">
-    <origin xyz="-0.18673 -0.066896 0.51747" rpy="0 0 0"/>
+    <origin xyz="-0.18673 -0.066898 0.75053" rpy="0 0 0"/>
     <parent link="base_link"/>
     <child  link="cam_stand_Link"/>
@@ -408,6 +408,6 @@
     <mu2>0.05</mu2>
     <fdir1>1 0 0</fdir1>
-    <kp>100000.0</kp>
-    <kd>100.0</kd>
+    <kp>10000000.0</kp>
+    <kd>1.0</kd>
     <minDepth>0.001</minDepth>
   </gazebo>
@@ -416,6 +416,6 @@
     <mu2>0.05</mu2>
     <fdir1>1 0 0</fdir1>
-    <kp>100000.0</kp>
-    <kd>100.0</kd>
+    <kp>10000000.0</kp>
+    <kd>1.0</kd>
     <minDepth>0.001</minDepth>
   </gazebo>
@@ -424,6 +424,6 @@
     <mu2>0.05</mu2>
     <fdir1>1 0 0</fdir1>
-    <kp>100000.0</kp>
-    <kd>100.0</kd>
+    <kp>10000000.0</kp>
+    <kd>1.0</kd>
     <minDepth>0.001</minDepth>
   </gazebo>
@@ -432,6 +432,6 @@
     <mu2>0.05</mu2>
     <fdir1>1 0 0</fdir1>
-    <kp>100000.0</kp>
-    <kd>100.0</kd>
+    <kp>10000000.0</kp>
+    <kd>1.0</kd>
     <minDepth>0.001</minDepth>
   </gazebo>
@@ -444,5 +444,5 @@
       <topic>lidar</topic>
       <gz_frame_id>laser_Link</gz_frame_id>
-      <update_rate>20</update_rate>
+      <update_rate>5</update_rate>
       <ray>
         <scan>
@@ -472,5 +472,5 @@
       </ray>
       <always_on>1</always_on>
-      <visualize>true</visualize>
+      <visualize>false</visualize>
     </sensor>
   </gazebo>
@@ -592,24 +592,3 @@
     </sensor>
   </gazebo>
-  <!-- ================================================================
-       THERMAL PROPERTIES — required for thermal camera sensor
-  ================================================================ -->
-  <gazebo reference="base_link">
-    <temperature>310.0</temperature>
-  </gazebo>
-  <gazebo reference="F_R_W_Link">
-    <temperature>305.0</temperature>
-  </gazebo>
-  <gazebo reference="F_L_W_Link">
-    <temperature>305.0</temperature>
-  </gazebo>
-  <gazebo reference="B_R_W_Link">
-    <temperature>305.0</temperature>
-  </gazebo>
-  <gazebo reference="B_L_W_Link">
-    <temperature>305.0</temperature>
-  </gazebo>
-  <gazebo reference="laser_Link">
-    <temperature>308.0</temperature>
-  </gazebo>
 </robot>

Commit message: feat: add camera stand trajectory control

File: src/amr_ix1_description/urdf/amr_ix1.urdf.xacro (robot description, xacro)
@@ -277,5 +277,5 @@
     <child  link="cam_stand_Link"/>
     <axis xyz="0 1 0"/>
-    <limit lower="-0.7854" upper="0" effort="10.0" velocity="1.5" />
+    <limit lower="-0.7854" upper="0.2" effort="10.0" velocity="1.5" />
     <dynamics damping="0.1" friction="0.1"/>
   </joint>
@@ -391,5 +391,5 @@
       <command_interface name="position">
         <param name="min">-0.7854</param>
-        <param name="max">0.0</param>
+        <param name="max">0.2</param>
       </command_interface>
       <state_interface name="position"/>

Commit message: Split URDF into modular xacro files with hardware/use_thermal switches

File: src/amr_ix1_description/urdf/amr_ix1.urdf.xacro (robot description, xacro)
@@ -2,597 +2,20 @@
 <robot xmlns:xacro="http://www.ros.org/wiki/xacro" name="amr_ix1">
   <!-- ================================================================
-       AMR-IX1 Inspection Robot — URDF/Xacro Description
+       AMR-IX1 Inspection Robot — top-level URDF/Xacro
        Maintainer: Hossam
        License: Apache-2.0
+       Arguments (defaults keep the old behaviour = Ignition simulation):
+         hardware     sim | mock | real      (default: sim)
+         use_thermal  true | false           (default: true; simulation only)
+       Example:  xacro amr_ix1.urdf.xacro hardware:=mock
   ================================================================ -->
-  <!-- ── Materials ────────────────────────────────────────────────── -->
-  <material name="dark_grey">
-    <color rgba="0.251 0.251 0.251 1.0"/>
-  </material>
-  <material name="light_grey">
-    <color rgba="0.753 0.753 0.753 1.0"/>
-  </material>
-  <material name="metal_grey">
-    <color rgba="0.627 0.627 0.627 1.0"/>
-  </material>
-  <material name="dark_charcoal">
-    <color rgba="0.212 0.212 0.204 1.0"/>
-  </material>
-  <material name="white">
-    <color rgba="1.0 0.984 0.984 1.0"/>
-  </material>
-  <material name="blue_grey">
-    <color rgba="0.792 0.820 0.933 1.0"/>
-  </material>
-  <!-- ================================================================
-       BASE FOOTPRINT — dummy root link (required by Nav2 and Gazebo)
-  ================================================================ -->
-  <link name="base_footprint"/>
-  <joint name="base_footprint_joint" type="fixed">
-    <origin xyz="0 0 0.3347" rpy="0 0 0"/>
-    <parent link="base_footprint"/>
-    <child  link="base_link"/>
-  </joint>
-  <!-- ================================================================
-       BASE LINK
-  ================================================================ -->
-  <link name="base_link">
-    <inertial>
-      <origin xyz="0.0 0.0 0.0" rpy="0 0 0"/>
-      <mass value="17.7024"/>
-      <inertia
-        ixx="0.212987" ixy="-4.778E-07" ixz="0.014399"
-        iyy="0.266448"  iyz="0.002175"
-        izz="0.358088"/>
-    </inertial>
-    <visual>
-      <origin xyz="0 0 0" rpy="0 0 0"/>
-      <geometry>
-        <mesh filename="package://amr_ix1_description/meshes/visual/base_link.STL"/>
-      </geometry>
-      <material name="dark_grey"/>
-    </visual>
-    <collision>
-      <origin xyz="0.10 0 0.11" rpy="0 0 0"/>
-      <geometry>
-        <box size="0.90 0.75 0.25"/>
-      </geometry>
-    </collision>
-  </link>
-  <!-- ================================================================
-       FRONT RIGHT WHEEL
-  ================================================================ -->
-  <link name="F_R_W_Link">
-    <inertial>
-      <origin rpy="0 0 0" xyz="0 0 0"/>
-      <mass value="1.5"/>
-      <inertia ixx="0.0029" ixy="0.0" ixz="0.0" iyy="0.0029" iyz="0.0" izz="0.0042"/>
-    </inertial>
-    <visual>
-      <origin xyz="0 0 0" rpy="0 0 0"/>
-      <geometry>
-        <mesh filename="package://amr_ix1_description/meshes/visual/F_R_W_Link.STL"/>
-              <scale>0.001 0.001 0.001</scale>
-      </geometry>
-      <material name="light_grey"/>
-    </visual>
-    <collision>
-	  <origin xyz="0 -0.025 0" rpy="1.5708 0 0"/>
-	  <geometry>
-	    <cylinder radius="0.155" length="0.12"/>
-	  </geometry>
-    </collision>
-  </link>
-  <joint name="F_R_W_joint" type="continuous">
-    <origin xyz="0.36 -0.45 -0.0300" rpy="0 0 0"/>
-    <parent link="base_link"/>
-    <child  link="F_R_W_Link"/>
-    <axis xyz="0 1 0"/>
-    <dynamics damping="3.0" friction="2.0"/>
-  </joint>
-  <!-- ================================================================
-       FRONT LEFT WHEEL
-  ================================================================ -->
-  <link name="F_L_W_Link">
-    <inertial>
-      <origin rpy="0 0 0" xyz="0 0 0"/>
-      <mass value="1.5"/>
-      <inertia ixx="0.0029" ixy="0.0" ixz="0.0" iyy="0.0029" iyz="0.0" izz="0.0042"/>
-    </inertial>
-    <visual>
-      <origin xyz="0 0 0" rpy="0 0 0"/>
-      <geometry>
-        <mesh filename="package://amr_ix1_description/meshes/visual/F_L_W_Link.STL"/>
-              <scale>0.001 0.001 0.001</scale>
-      </geometry>
-      <material name="light_grey"/>
-    </visual>
-    <collision>
-	  <origin xyz="0 0.025 0" rpy="1.5708 0 0"/>
-	  <geometry>
-	    <cylinder radius="0.155" length="0.12"/>
-	  </geometry>
-    </collision>
-  </link>
-  <joint name="F_L_W_joint" type="continuous">
-    <origin xyz="0.36 0.45 -0.0300" rpy="0 0 0"/>
-    <parent link="base_link"/>
-    <child  link="F_L_W_Link"/>
-    <axis xyz="0 1 0"/>
-    <dynamics damping="3.0" friction="2.0"/>
-  </joint>
-  <!-- ================================================================
-       BACK RIGHT WHEEL
-  ================================================================ -->
-  <link name="B_R_W_Link">
-    <inertial>
-      <origin rpy="0 0 0" xyz="0 0 0"/>
-      <mass value="1.5"/>
-      <inertia ixx="0.0029" ixy="0.0" ixz="0.0" iyy="0.0029" iyz="0.0" izz="0.0042"/>
-    </inertial>
-    <visual>
-      <origin xyz="0 0 0" rpy="0 0 0"/>
-      <geometry>
-        <mesh filename="package://amr_ix1_description/meshes/visual/B_R_W_Link.STL"/>
-              <scale>0.001 0.001 0.001</scale>
-      </geometry>
-      <material name="light_grey"/>
-    </visual>
-    <collision>
-	  <origin xyz="0 -0.025 0" rpy="1.5708 0 0"/>
-	  <geometry>
-	    <cylinder radius="0.155" length="0.12"/>
-	  </geometry>
-    </collision>
-  </link>
-  <joint name="B_R_W_joint" type="continuous">
-    <origin xyz="-0.36 -0.45 -0.0300" rpy="0 0 0"/>
-    <parent link="base_link"/>
-    <child  link="B_R_W_Link"/>
-    <axis xyz="0 1 0"/>
-    <dynamics damping="3.0" friction="2.0"/>
-  </joint>
-  <!-- ================================================================
-       BACK LEFT WHEEL
-  ================================================================ -->
-  <link name="B_L_W_Link">
-    <inertial>
-      <origin rpy="0 0 0" xyz="0 0 0"/>
-      <mass value="1.5"/>
-      <inertia ixx="0.0029" ixy="0.0" ixz="0.0" iyy="0.0029" iyz="0.0" izz="0.0042"/>
-    </inertial>
-    <visual>
-      <origin xyz="0 0 0" rpy="0 0 0"/>
-      <geometry>
-        <mesh filename="package://amr_ix1_description/meshes/visual/B_L_W_Link.STL"/>
-              <scale>0.001 0.001 0.001</scale>
-      </geometry>
-      <material name="light_grey"/>
-    </visual>
-    <collision>
-	  <origin xyz="0 0.025 0" rpy="1.5708 0 0"/>
-	  <geometry>
-	    <cylinder radius="0.155" length="0.12"/>
-	  </geometry>
-    </collision>
-  </link>
-  <joint name="B_L_W_joint" type="continuous">
-    <origin xyz="-0.36 0.45 -0.0300" rpy="0 0 0"/>
-    <parent link="base_link"/>
-    <child  link="B_L_W_Link"/>
-    <axis xyz="0 1 0"/>
-    <dynamics damping="3.0" friction="2.0"/>
-  </joint>
-  <!-- ================================================================
-       IMU
-  ================================================================ -->
-  <link name="imu_Link">
-    <inertial>
-      <origin xyz="-0.000400 0.000132 0.006812" rpy="0 0 0"/>
-      <mass value="0.010837"/>
-      <inertia
-        ixx="9.951E-07" ixy="2.081E-08" ixz="1.091E-08"
-        iyy="9.555E-07"  iyz="-3.252E-09"
-        izz="1.642E-06"/>
-    </inertial>
-    <visual>
-      <origin xyz="0 0 0" rpy="3.14159 0 0"/>
-      <geometry>
-        <mesh filename="package://amr_ix1_description/meshes/visual/imu_Link.STL"/>
-      </geometry>
-      <material name="metal_grey"/>
-    </visual>
-    <collision>
-      <origin xyz="0 0 0" rpy="3.14159 0 0"/>
-      <geometry>
-        <mesh filename="package://amr_ix1_description/meshes/collision/imu_Link.STL"/>
-      </geometry>
-    </collision>
-  </link>
-  <joint name="imu_joint" type="fixed">
-    <origin xyz="0.0 0.0 0.0" rpy="0 0 0"/>
-    <parent link="base_link"/>
-    <child  link="imu_Link"/>
-  </joint>
-  <!-- ================================================================
-       LIDAR
-  ================================================================ -->
-  <link name="laser_Link">
-    <inertial>
-      <origin xyz="-0.005720 0.001226 -0.009051" rpy="0 0 0"/>
-      <mass value="0.141654"/>
-      <inertia
-        ixx="5.691E-05" ixy="-2.879E-07" ixz="-1.248E-05"
-        iyy="8.932E-05"  iyz="7.219E-07"
-        izz="1.087E-04"/>
-    </inertial>
-    <visual>
-      <origin xyz="0 0 0" rpy="0 0 0"/>
-      <geometry>
-        <mesh filename="package://amr_ix1_description/meshes/visual/laser_Link.STL"/>
-      </geometry>
-      <material name="dark_charcoal"/>
-    </visual>
-    <collision>
-      <origin xyz="0 0 0" rpy="0 0 0"/>
-      <geometry>
-        <mesh filename="package://amr_ix1_description/meshes/collision/laser_Link.STL"/>
-      </geometry>
-    </collision>
-  </link>
-  <joint name="laser_joint" type="fixed">
-    <origin xyz="0.415447680695362 -0.00758871084657819 0.27756000072765" rpy="0 0 0"/>
-    <parent link="base_link"/>
-    <child  link="laser_Link"/>
-  </joint>
-  <!-- ================================================================
-       CAMERA STAND
-  ================================================================ -->
-  <link name="cam_stand_Link">
-    <inertial>
-      <origin xyz="0.005597 0.032884 -0.000945" rpy="0 0 0"/>
-      <mass value="0.008532"/>
-      <inertia
-        ixx="5.125E-06" ixy="-1.127E-07" ixz="2.108E-09"
-        iyy="9.300E-07"  iyz="1.718E-08"
-        izz="4.259E-06"/>
-    </inertial>
-    <visual>
-      <origin xyz="0 0 0" rpy="0 0 0"/>
-      <geometry>
-        <mesh filename="package://amr_ix1_description/meshes/visual/cam_stand_Link.STL"/>
-      </geometry>
-      <material name="blue_grey"/>
-    </visual>
-    <collision>
-      <origin xyz="0 0 0" rpy="0 0 0"/>
-      <geometry>
-        <mesh filename="package://amr_ix1_description/meshes/collision/cam_stand_Link.STL"/>
-      </geometry>
-    </collision>
-  </link>
-  <joint name="cam_stand_joint" type="revolute">
-    <origin xyz="-0.18673 -0.066898 0.75053" rpy="0 0 0"/>
-    <parent link="base_link"/>
-    <child  link="cam_stand_Link"/>
-    <axis xyz="0 1 0"/>
-    <limit lower="-0.7854" upper="0.2" effort="10.0" velocity="1.5" />
-    <dynamics damping="0.1" friction="0.1"/>
-  </joint>
-  <!-- ================================================================
-       CAMERA
-  ================================================================ -->
-  <link name="camera_Link">
-    <inertial>
-      <origin xyz="-0.010605 -5.056E-05 -0.001198" rpy="0 0 0"/>
-      <mass value="0.025772"/>
-      <inertia
-        ixx="6.271E-06" ixy="1.006E-11" ixz="3.897E-09"
-        iyy="4.255E-06"  iyz="1.509E-10"
-        izz="4.285E-06"/>
-    </inertial>
-    <visual>
-      <origin xyz="0 0 0" rpy="0 0 0"/>
-      <geometry>
-        <mesh filename="package://amr_ix1_description/meshes/visual/camera_Link.STL"/>
-      </geometry>
-      <material name="white"/>
-    </visual>
-    <collision>
-      <origin xyz="0 0 0" rpy="0 0 0"/>
-      <geometry>
-        <mesh filename="package://amr_ix1_description/meshes/collision/camera_Link.STL"/>
-      </geometry>
-    </collision>
-  </link>
-  <joint name="camera_joint" type="fixed">
-    <origin xyz="0.028695 0.053607 0.000157" rpy="0 0 0"/>
-    <parent link="cam_stand_Link"/>
-    <child  link="camera_Link"/>
-  </joint>
-  <!-- ================================================================
-       THERMAL CAMERA
-  ================================================================ -->
-  <link name="thermal_link">
-    <inertial>
-      <origin xyz="-0.009412 0.000127 -0.000586" rpy="0 0 0"/>
-      <mass value="0.024852"/>
-      <inertia
-        ixx="6.238E-06" ixy="1.086E-11" ixz="3.867E-09"
-        iyy="4.239E-06"  iyz="-6.644E-11"
-        izz="4.273E-06"/>
-    </inertial>
-    <visual>
-      <origin xyz="0 0 0" rpy="0 0 0"/>
-      <geometry>
-        <mesh filename="package://amr_ix1_description/meshes/visual/thermal_link.STL"/>
-      </geometry>
-      <material name="blue_grey"/>
-    </visual>
-    <collision>
-      <origin xyz="0 0 0" rpy="0 0 0"/>
-      <geometry>
-        <mesh filename="package://amr_ix1_description/meshes/collision/thermal_link.STL"/>
-      </geometry>
-    </collision>
-  </link>
-  <joint name="thermal_joint" type="fixed">
-    <origin xyz="0.027189 0.016420 -0.000526" rpy="0 0 0"/>
-    <parent link="cam_stand_Link"/>
-    <child  link="thermal_link"/>
-  </joint>
-  <!-- ================================================================
-       ROS2 CONTROL — Hardware Interface
-       Uses ign_ros2_control for Gazebo simulation
-       Same interface will be used for real hardware (ESP32)
-  ================================================================ -->
-  <ros2_control name="amr_ix1_system" type="system">
-    <hardware>
-      <plugin>ign_ros2_control/IgnitionSystem</plugin>
-    </hardware>
-    <!-- Front Right Wheel -->
-    <joint name="F_R_W_joint">
-      <command_interface name="velocity">
-        <param name="min">-10</param>
-        <param name="max">10</param>
-      </command_interface>
-      <state_interface name="position"/>
-      <state_interface name="velocity"/>
-    </joint>
-    <!-- Front Left Wheel -->
-    <joint name="F_L_W_joint">
-      <command_interface name="velocity">
-        <param name="min">-10</param>
-        <param name="max">10</param>
-      </command_interface>
-      <state_interface name="position"/>
-      <state_interface name="velocity"/>
-    </joint>
-    <!-- Back Right Wheel -->
-    <joint name="B_R_W_joint">
-      <command_interface name="velocity">
-        <param name="min">-10</param>
-        <param name="max">10</param>
-      </command_interface>
-      <state_interface name="position"/>
-      <state_interface name="velocity"/>
-    </joint>
-    <!-- Back Left Wheel -->
-    <joint name="B_L_W_joint">
-      <command_interface name="velocity">
-        <param name="min">-10</param>
-        <param name="max">10</param>
-      </command_interface>
-      <state_interface name="position"/>
-      <state_interface name="velocity"/>
-    </joint>
-    <!-- Camera Stand — position controlled -->
-    <joint name="cam_stand_joint">
-      <command_interface name="position">
-        <param name="min">-0.7854</param>
-        <param name="max">0.2</param>
-      </command_interface>
-      <state_interface name="position"/>
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